File: FlowerBed.kicad_pcb (KiCad board)
At the start: 2 copper layers, 121.3 x 110 mm, 28 parts, among them J1 Conn_01x02, J2 AudioJack3_SwitchTR, J3 AudioJack3_SwitchTR, J4 Conn_01x07, J5 Conn_01x16, J6 Conn_01x02, SW0 SW_SPST, SW1 SW_SPST, SW2 SW_SPST, SW3 SW_SPST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

Commit message: Begins alternate layout with pots above switches
Parts:
- moved POT0 35.6 mm to (42.0, 45.6)
- moved POT1 35.6 mm to (62.3, 45.6)
- moved POT2 35.6 mm to (82.6, 45.6)
- moved POT3 35.6 mm to (102.9, 45.6)
- moved SW0 21.7 mm to (50.8, 61.0)
- moved SW1 21.7 mm to (71.1, 61.0)
- moved SW2 21.7 mm to (91.4, 61.0)
- moved SW3 21.7 mm to (111.8, 61.0)
- moved SW4 21.7 mm to (50.8, 80.0)
- moved SW5 21.7 mm to (71.1, 80.0)
- moved SW6 21.7 mm to (91.4, 80.0)
- moved SW7 21.7 mm to (111.8, 80.0)
Routing:
- net /3V3_A: track 140.5 -> 16.5 mm, vias 3 -> 0
- net /D15_A0: track 114.1 -> 14.3 mm, vias 4 -> 0
- net /D16_A1: track 92.5 -> 12.2 mm, vias 4 -> 0
- net /D4: track 78.7 -> 12.5 mm
- net /D0: track 77.9 -> 13.6 mm
- net /D17_A2: track 71.1 -> 9.12 mm, vias 4 -> 0
- net /D18_A3: track 50.5 -> 6.05 mm, vias 4 -> 0
- net /D5: track 58.1 -> 14.3 mm
- net /D1: track 56.8 -> 14.1 mm
- net /D2: track 36.5 -> 14.6 mm
- net /D3: track 14.1 -> 32.7 mm
- net /D6: track 36.0 -> 25.0 mm
- net /D7: track 14.6 -> 23.2 mm
Other:
- outline, holes or cut-outs redrawn
- board text removed: "A0"
- board text removed: "A1"
- board text removed: "A2"
- board text removed: "A3"

Commit message: Legacy active sum
Parts:
- POT0, POT1, POT2, POT3: footprint FlowerbedLib:Potentiometer_LMS -> Potentiometer_THT:Potentiometer_Alpha_RD901F-40-00D_Single_Vertical
- moved POT0 61.0 mm to (102.9, 48.1)
- moved POT3 61.0 mm to (42.0, 48.1)
- moved POT1 20.5 mm to (82.6, 48.1)
- moved POT2 20.5 mm to (62.3, 48.1)
- moved SW0 2.54 mm to (50.8, 63.5)
- moved SW1 2.54 mm to (71.1, 63.5)
- moved SW2 2.54 mm to (91.4, 63.5)
- moved SW3 2.54 mm to (111.8, 63.5)
- moved SW4 2.54 mm to (50.8, 82.5)
- moved SW5 2.54 mm to (71.1, 82.5)
- moved SW6 2.54 mm to (91.4, 82.5)
- moved SW7 2.54 mm to (111.8, 82.5)
Routing:
- net /3V3_A: track 16.5 -> 269.7 mm, vias 0 -> 8
- net /D18_A3: track 6.05 -> 155.4 mm
- net /D17_A2: track 9.12 -> 135.1 mm, vias 0 -> 2
- net /D16_A1: track 12.2 -> 114.1 mm, vias 0 -> 2
- net /D0: track 13.6 -> 100.0 mm
- net /D4: track 12.5 -> 98.4 mm
- net /D1: track 14.1 -> 94.3 mm
- net /D15_A0: track 14.3 -> 93.3 mm, vias 0 -> 2
- net /D5: track 14.3 -> 77.0 mm
- net /D2: track 14.6 -> 57.9 mm
- net /D6: track 25.0 -> 55.7 mm
- net /D3: track 32.7 -> 52.2 mm
- net /D7: track 23.2 -> 40.2 mm
Other:
- outline, holes or cut-outs redrawn
- board text added: "A0"
- board text added: "A1"
- board text added: "A2"
- board text added: "A3"
